File: Criticality/criticality_shield.brd (EAGLE design)
At the start: 100 x 80.5 mm, 73 parts

Commit message: before groundplates
Parts:
- moved D22-36_EVEN 0.25 mm to (68.0, 41.2)
- moved D23-37-ODD 0.25 mm to (70.5, 41.2)
- moved D38-52-EVEN 0.25 mm to (68.0, 18.8)
- moved D39-53-ODD 0.25 mm to (70.5, 18.8)
Routing:
- net GND: track 228.7 -> 226.8 mm

Commit message: final
Routing:
- added copper zone on layer 1, net GND
- added copper zone on layer 16, net GND
Changed lines of the file:
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@@
 <wire x1="57" y1="23.5" x2="52" y2="23.5" width="0.254" layer="16"/>
 <wire x1="68.1228" y1="8.4582" x2="68" y2="8.4582" width="0.4064" layer="1"/>
-<wire x1="68" y1="8.4582" x2="68" y2="8.5" width="0" layer="19" extent="1-16"/>
 <via x="62.4506" y="58.0216" extent="1-16" drill="0.6" shape="square"/>
-<wire x1="68" y1="8.5" x2="68" y2="6" width="0" layer="19" extent="1-16"/>
 <wire x1="68" y1="8.5" x2="68" y2="5.5" width="0.254" layer="1"/>
 <via x="68" y="5.5" extent="1-16" drill="0.6" shape="square"/>
@@
 <wire x1="52" y1="24.5" x2="17.5" y2="24.5" width="0.254" layer="16"/>
 <wire x1="17.5" y1="24.5" x2="17.5" y2="38.5" width="0.254" layer="16"/>
+<polygon width="0.4064" layer="16" isolate="0.254">
+<vertex x="0" y="80.5"/>
+<vertex x="0" y="0"/>
+<vertex x="100" y="0"/>
+<vertex x="100" y="1.5"/>
+<vertex x="100" y="80.5"/>
+</polygon>
+<polygon width="0.4064" layer="1" isolate="0.254">
+<vertex x="0" y="80.5"/>
+<vertex x="0" y="-0.5"/>
+<vertex x="100" y="-0.5"/>
+<vertex x="100" y="3.5"/>
+<vertex x="100" y="81"/>
+<vertex x="0" y="81"/>
+</polygon>
 </signal>
 <signal name="+5V">
@@
 <wire x1="36.8046" y1="43.434" x2="36.73" y2="43.6" width="0.254" layer="1"/>
 <wire x1="36.8046" y1="41.148" x2="36.73" y2="41.06" width="0.254" layer="1"/>
-<wire x1="44.8056" y1="21.717" x2="47.5488" y2="21.717" width="0.254" layer="1"/>
-<wire x1="43.2054" y1="23.3172" x2="44.8056" y2="21.717" width="0.254" layer="1"/>
+<wire x1="44.8056" y1="21.217" x2="47.5488" y2="21.217" width="0.254" layer="1"/>
+<wire x1="43.2054" y1="23.3172" x2="44.8056" y2="21.217" width="0.254" layer="1"/>
 <wire x1="41.3766" y1="23.3172" x2="43.2054" y2="23.3172" width="0.254" layer="1"/>
 <wire x1="40.2336" y1="22.1742" x2="41.3766" y2="23.3172" width="0.254" layer="1"/>
-<wire x1="47.5488" y1="21.717" x2="47.5978" y2="21.525" width="0.254" layer="1"/>
+<wire x1="47.5488" y1="21.217" x2="47.5978" y2="21.525" width="0.254" layer="1"/>
 <wire x1="40.2336" y1="22.1742" x2="40.23" y2="22.14" width="0.254" layer="1"/>
 <wire x1="40.2336" y1="21.9456" x2="40.2336" y2="19.6596" width="0.254" layer="1"/>
@@
 <contactref element="ULN5" pad="7"/>
 <wire x1="62.6364" y1="25.146" x2="62.6364" y2="25.8318" width="0.254" layer="1"/>
-<wire x1="59.2074" y1="21.717" x2="62.6364" y2="25.146" width="0.254" layer="1"/>
-<wire x1="59.2074" y1="20.1168" x2="59.2074" y2="21.717" width="0.254" layer="1"/>
+<wire x1="60.7074" y1="24.217" x2="62.6364" y2="25.146" width="0.254" layer="1"/>
+<wire x1="59.2074" y1="20.1168" x2="60.7074" y2="24.217" width="0.254" layer="1"/>
 <wire x1="58.293" y1="19.2024" x2="59.2074" y2="20.1168" width="0.254" layer="1"/>
 <wire x1="57.6072" y1="19.2024" x2="58.293" y2="19.2024" width="0.254" layer="1"/>
@@
 <contactref element="JP6" pad="3"/>
 <wire x1="46.863" y1="12.573" x2="47.5488" y2="12.573" width="0.254" layer="1"/>
-<wire x1="43.8912" y1="9.6012" x2="46.863" y2="12.573" width="0.254" layer="1"/>
-<wire x1="43.8912" y1="8.001" x2="43.8912" y2="9.6012" width="0.254" layer="1"/>
+<wire x1="44.3912" y1="10.1012" x2="46.863" y2="12.573" width="0.254" layer="1"/>
+<wire x1="43.8912" y1="8.001" x2="44.3912" y2="10.1012" width="0.254" layer="1"/>
 <wire x1="42.9768" y1="7.0866" x2="43.8912" y2="8.001" width="0.254" layer="1"/>
 <wire x1="47.5488" y1="12.573" x2="47.5978" y2="12.635" width="0.254" layer="1"/>
@@
 <contactref element="ULN5" pad="13"/>
 <contactref element="JP6" pad="11"/>
-<wire x1="43.434" y1="17.6022" x2="47.5488" y2="17.6022" width="0.254" layer="1"/>
-<wire x1="42.9768" y1="17.145" x2="43.434" y2="17.6022" width="0.254" layer="1"/>
-<wire x1="47.5488" y1="17.6022" x2="47.5978" y2="17.715" width="0.254" layer="1"/>
+<wire x1="42.934" y1="17.6022" x2="47.0488" y2="17.6022" width="0.254" layer="1"/>
+<wire x1="42.9768" y1="17.145" x2="42.934" y2="17.6022" width="0.254" layer="1"/>
+<wire x1="47.0488" y1="17.6022" x2="47.5978" y2="17.715" width="0.254" layer="1"/>
 <wire x1="42.9768" y1="17.145" x2="42.77" y2="17.06" width="0.254" layer="1"/>
 </signal>
@@
 <contactref element="ULN5" pad="12"/>
 <contactref element="JP6" pad="13"/>
-<wire x1="43.2054" y1="19.2024" x2="47.5488" y2="19.2024" width="0.254" layer="1"/>
-<wire x1="42.9768" y1="19.431" x2="43.2054" y2="19.2024" width="0.254" layer="1"/>
-<wire x1="47.5488" y1="19.2024" x2="47.5978" y2="18.985" width="0.254" layer="1"/>
+<wire x1="42.7054" y1="19.2024" x2="47.0488" y2="19.2024" width="0.254" layer="1"/>
+<wire x1="42.9768" y1="19.431" x2="42.7054" y2="19.2024" width="0.254" layer="1"/>
+<wire x1="47.0488" y1="19.2024" x2="47.5978" y2="18.985" width="0.254" layer="1"/>
 <wire x1="42.9768" y1="19.431" x2="42.77" y2="19.6" width="0.254" layer="1"/>
 </signal>
