File: Criticality/criticality_shield.sch (EAGLE design)
At the start: 73 parts

Commit message: further improvements
Changed lines of the file:
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@@
 <part name="R13" library="SparkFun-Resistors" deviceset="RESISTOR" device="0603"/>
 <part name="R14" library="SparkFun-Resistors" deviceset="RESISTOR" device="0603"/>
-<part name="GND9" library="supply1" deviceset="GND" device=""/>
-<part name="SUPPLY17" library="supply2" deviceset="+5V" device=""/>
 <part name="ULN2" library="SparkFun-PowerIC" deviceset="ULN2803" device="SOICW"/>
 <part name="R15" library="SparkFun-Resistors" deviceset="RESISTOR" device="0603"/>
@@
 <instance part="GND2" gate="1" x="-50.8" y="132.08"/>
 <instance part="D0-7" gate="1" x="-66.04" y="157.48" rot="R180"/>
-<instance part="GND1" gate="1" x="-48.26" y="73.66"/>
+<instance part="GND1" gate="1" x="-50.8" y="73.66"/>
 <instance part="D14-21" gate="1" x="30.48" y="167.64" rot="R180"/>
 <instance part="GND3" gate="1" x="53.34" y="132.08"/>
@@
 <instance part="SUPPLY2" gate="+5V" x="114.3" y="152.4"/>
 <instance part="SUPPLY5" gate="+5V" x="81.28" y="132.08" rot="R180"/>
-<instance part="SUPPLY6" gate="+5V" x="-15.24" y="73.66" rot="R180"/>
+<instance part="SUPPLY6" gate="+5V" x="-17.78" y="73.66" rot="R180"/>
 <instance part="SUPPLY7" gate="+5V" x="-12.7" y="132.08" rot="R180"/>
 <instance part="JP1" gate="A" x="-5.08" y="162.56"/>
@@
 <instance part="R13" gate="G$1" x="43.18" y="175.26"/>
 <instance part="R14" gate="G$1" x="43.18" y="180.34"/>
-<instance part="GND9" gate="1" x="-48.26" y="73.66"/>
-<instance part="SUPPLY17" gate="+5V" x="-15.24" y="73.66" rot="R180"/>
 <instance part="ULN2" gate="G$1" x="-33.02" y="104.14"/>
 <instance part="R15" gate="G$1" x="-55.88" y="111.76"/>
@@
 <segment>
 <pinref part="GND1" gate="1" pin="GND"/>
-<wire x1="-45.72" y1="76.2" x2="-48.26" y2="76.2" width="0.1524" layer="91"/>
-<junction x="-48.26" y="76.2"/>
+<wire x1="-50.8" y1="76.2" x2="-45.72" y2="76.2" width="0.1524" layer="91"/>
+<pinref part="ULN2" gate="G$1" pin="9"/>
+<wire x1="-45.72" y1="81.28" x2="-45.72" y2="76.2" width="0.1524" layer="91"/>
+<junction x="-45.72" y="81.28"/>
+<junction x="-45.72" y="76.2"/>
+<junction x="-50.8" y="76.2"/>
 </segment>
 <segment>
@@
 <pinref part="GND3" gate="1" pin="GND"/>
 <junction x="53.34" y="134.62"/>
-</segment>
-<segment>
-<pinref part="GND9" gate="1" pin="GND"/>
-<wire x1="-48.26" y1="76.2" x2="-45.72" y2="76.2" width="0.1524" layer="91"/>
-<junction x="-48.26" y="76.2"/>
-<pinref part="ULN2" gate="G$1" pin="9"/>
-<wire x1="-45.72" y1="81.28" x2="-45.72" y2="76.2" width="0.1524" layer="91"/>
-<junction x="-45.72" y="81.28"/>
 </segment>
 <segment>
@@
 <segment>
 <pinref part="SUPPLY6" gate="+5V" pin="+5V"/>
-<wire x1="-17.78" y1="76.2" x2="-15.24" y2="76.2" width="0.1524" layer="91"/>
-<junction x="-15.24" y="76.2"/>
+<pinref part="ULN2" gate="G$1" pin="10"/>
+<wire x1="-17.78" y1="81.28" x2="-17.78" y2="76.2" width="0.1524" layer="91"/>
+<junction x="-17.78" y="81.28"/>
+<junction x="-17.78" y="76.2"/>
 </segment>
 <segment>
@@
 </segment>
 <segment>
-<pinref part="SUPPLY17" gate="+5V" pin="+5V"/>
-<wire x1="-17.78" y1="76.2" x2="-15.24" y2="76.2" width="0.1524" layer="91"/>
-<junction x="-15.24" y="76.2"/>
-<pinref part="ULN2" gate="G$1" pin="10"/>
-<wire x1="-17.78" y1="81.28" x2="-17.78" y2="76.2" width="0.1524" layer="91"/>
-<junction x="-17.78" y="81.28"/>
-</segment>
-<segment>
 <pinref part="ULN1" gate="G$1" pin="10"/>
 <pinref part="SUPPLY7" gate="+5V" pin="+5V"/>
@@
 </segment>
 </net>
-<net name="N$17" class="0">
-<segment>
-<wire x1="-17.78" y1="63.5" x2="-7.62" y2="60.96" width="0.1524" layer="91"/>
-</segment>
-</net>
 <net name="N$133" class="0">
 <segment>
@@
 </sheet>
 </sheets>
+<errors>
+</errors>
 </schematic>
 </drawing>
