File: Criticality/criticality_shield_improved.sch (EAGLE design)
At the start: 74 parts, among them U1 ARDUINO-MEGAFULL

Commit message: -
Parts:
- removed U1: ARDUINO-MEGAFULL, SparkFun-Boards:ARDUINO-MEGAFULL
Changed lines of the file:
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@@
 <part name="JP9" library="pinhead" deviceset="PINHD-2X6" device=""/>
 <part name="SUPPLY9" library="supply2" deviceset="+5V" device=""/>
-<part name="U1" library="SparkFun-Boards" deviceset="ARDUINO-MEGA" device="FULL"/>
 </parts>
 <sheets>
@@
 <instance part="JP9" gate="A" x="-5.08" y="109.22"/>
 <instance part="SUPPLY9" gate="+5V" x="0" y="93.98" rot="R180"/>
-<instance part="U1" gate="G$1" x="40.64" y="45.72" rot="R90"/>
 </instances>
 <busses>
