File: E-meter/E-meter2.brd (EAGLE design)
At the start: 89.8 x 72.4 mm, 32 parts, among them IC1 LM324N, IC2 7805T

Commit message: new layout
Parts:
- R13, R14: value POT_US-EVUF2A -> POT_US-EVUF2M; device 4009dist_PWM3_v1:POT_EVUF -> 4009dist_PWM3_v1:POT_EVUFXM
- moved IC2 80.8 mm to (86.4, 43.2), turned to 270 degrees
- moved GND9V 72.1 mm to (81.3, 52.1)
- moved +9V 62.0 mm to (76.2, 52.1)
- moved R1 59.6 mm to (35.6, 69.8), turned to 270 degrees
- moved R14 59.6 mm to (24.1, 11.4), turned to 180 degrees
- moved R8 58.2 mm to (33.0, 69.8), turned to 270 degrees
- moved R3 55.5 mm to (38.1, 69.8), turned to 90 degrees
- moved R9 44.5 mm to (20.3, 25.4)
- moved E2 40.0 mm to (76.2, 16.5), turned to 0 degrees
- moved R5 39.7 mm to (85.1, 16.5), turned to 0 degrees
- moved R12 39.6 mm to (63.5, 38.1), turned to 0 degrees
- moved E1 38.8 mm to (31.8, 48.3), turned to 0 degrees
- moved LED1 38.3 mm to (24.1, 69.8), turned to 0 degrees
- moved R15 38.2 mm to (15.2, 69.8), turned to 180 degrees
- moved R6 37.6 mm to (85.1, 19.1), turned to 0 degrees
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Connections:
- new net N$18: GND9V.1
- net GND: no longer GND9V.1
Routing:
- net N$15: track 137.9 -> 28.6 mm
- net N$4: track 96.7 -> 156.2 mm
- net N$17: track 81.0 -> 22.3 mm
- net N$6: track 70.6 -> 12.7 mm
- net GND: track 0.00 -> 53.3 mm
- net N$14: track 44.0 -> 86.4 mm
- net N$20: track 11.3 -> 46.5 mm
- net N$7: track 41.2 -> 6.35 mm
- net N$21: track 26.4 -> 3.20 mm
- net N$8: track 24.0 -> 2.54 mm
- net N$24: track 23.5 -> 6.43 mm
- net N$22: track 21.0 -> 5.08 mm
- net N$16: track 20.5 -> 7.70 mm
- net N$11: track 11.6 -> 17.8 mm
- net N$12: track 17.4 -> 22.9 mm
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Other:
- board size 89.8 x 72.4 mm -> 100 x 80 mm

Commit message: new files last version, hand corrected pdf
Parts:
- D1, D2, D3, D4: device diode:DO35-10 -> studioalgorhythmics_parts:DO35-10
- IC1: device linear:DIL14 -> studioalgorhythmics_parts:DIL14
- LED1: device SparkFun-LED:LED5MM -> studioalgorhythmics_parts:LED5MM
- PRESET1, PRESET2, PRESET3, PRESET4: device dp_devices:TRIMMER_3306F -> studioalgorhythmics_parts:TRIMMER_3306F
- R1, R10, R11, R12, R15, R2, R3, R4, R5, R6, R7, R8, R9: device rcl:0207/10 -> studioalgorhythmics_parts:0207/10
- R13, R14: device 4009dist_PWM3_v1:POT_EVUFXM -> studioalgorhythmics_parts:POT_EVUFXM
- moved GND 16.7 mm to (12.3, 25.0)
- moved MT 7.76 mm to (12.3, 30.6)
- moved D2 6.48 mm to (15.5, 40.5)
- moved D1 4.59 mm to (15.9, 55.8)
- moved R8 3.87 mm to (29.5, 68.3)
- moved R10 1.85 mm to (31.2, 38.9)
- moved R12 1.78 mm to (63.5, 36.3)
- moved R2 1.59 mm to (29.7, 55.8)
- moved R5 1.52 mm to (85.1, 15.0)
- moved E2 1.40 mm to (76.1, 15.1)
- moved R3 1.27 mm to (39.4, 69.8)
- moved D4 1.14 mm to (9.02, 40.6)
- moved R11 1.14 mm to (54.7, 45.7)
- moved R15 1.14 mm to (14.1, 69.8)
- moved R4 0.52 mm to (41.4, 31.6)
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Routing:
- net N$10: track 2.54 -> 15.6 mm
- net N$11: track 17.8 -> 11.5 mm
- net N$4: track 156.2 -> 150.9 mm
- net N$22: track 5.08 -> 10.1 mm
- net N$1: track 19.7 -> 16.0 mm
- net N$16: track 7.70 -> 4.37 mm
- net N$23: track 14.0 -> 17.1 mm
- net N$17: track 22.3 -> 20.5 mm
- net N$13: track 17.8 -> 16.1 mm
- net N$5: track 8.89 -> 10.3 mm
- net N$3: track 14.0 -> 12.7 mm
- net N$12: track 22.9 -> 24.1 mm
- net N$8: track 2.54 -> 3.68 mm
- net GND: track 53.3 -> 54.4 mm
- net N$26: track 2.54 -> 3.18 mm
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Other:
- board size 100 x 80 mm -> 100.1 x 80 mm

Commit message: last adjustments cleaning of last_fin not mirrored with Illustrator
Parts:
- moved R15 72.8 mm to (86.1, 59.2), turned to 0 degrees
- moved LED1 53.0 mm to (76.1, 59.2), turned to 180 degrees
- moved R3 17.2 mm to (54.1, 61.0)
- moved R1 9.67 mm to (44.7, 66.0), turned to 180 degrees
- moved R8 6.99 mm to (27.2, 61.7), turned to 0 degrees
Connections:
- net N$22: now also IC1.7; no longer R8.1
- net N$3: now also IC1.6, R8.2; no longer IC1.7
- net N$4: now also R8.1; no longer IC1.6, R8.2
Routing:
- net N$3: track 12.7 -> 61.3 mm
- net GND: track 54.4 -> 13.1 mm
- net N$14: track 85.9 -> 58.7 mm
- net N$22: track 10.1 -> 26.4 mm
- net N$4: track 150.9 -> 141.2 mm
- net N$5: track 10.3 -> 15.0 mm
- net N$2: track 18.8 -> 20.1 mm
